Commit message: update

File: src/autocar_description/urdf/autocar.xacro (robot description, xacro)
@@ -11,5 +11,5 @@
   <link name="base_link" />
   <joint name="chassis_link_joint" type="fixed">
-    <origin xyz="0 0 0.4936" rpy="0 0 0" />
+    <origin xyz="0 0 0.4936" rpy="0 0 -1.5708" />
     <parent link="base_link" />
     <child link="chassis_link" />

Commit message: update

File: src/autocar_description/urdf/autocar.xacro (robot description, xacro)
@@ -21,4 +21,41 @@
     <child link="hokuyo_link" />
   </joint>
+  <joint name="front_lidar_joint" type="fixed">
+    <origin xyz="0 0 0" rpy="0 0 0" />
+    <parent link="hokuyo_link" />
+    <child link="front_lidar_link" />
+  </joint>
+  <link name="front_lidar_link" />
+  <joint name="imu_joint" type="fixed">
+    <origin xyz="0 0 0.75" rpy="0 0 0" />
+    <parent link="base_link" />
+    <child link="imu_link" />
+  </joint>
+  <link name="imu_link">
+    <inertial>
+      <mass value="1e-5" />
+      <origin xyz="0 0 0" rpy="0 0 0" />
+      <inertia ixx="1e-6" ixy="0" ixz="0" iyy="1e-6" iyz="0" izz="1e-6" />
+    </inertial>
+  </link>
+  <joint name="front_camera_joint" type="fixed">
+    <origin xyz="2.20 0 1.10" rpy="0 0 0" />
+    <parent link="base_link" />
+    <child link="front_camera_link" />
+  </joint>
+  <link name="front_camera_link">
+    <visual>
+      <origin xyz="0 0 0" rpy="0 0 0" />
+      <geometry>
+        <box size="0.08 0.05 0.05" />
+      </geometry>
+      <material name="darkgrey" />
+    </visual>
+    <inertial>
+      <mass value="1e-5" />
+      <origin xyz="0 0 0" rpy="0 0 0" />
+      <inertia ixx="1e-6" ixy="0" ixz="0" iyy="1e-6" iyz="0" izz="1e-6" />
+    </inertial>
+  </link>
   <link name="hokuyo_link">
     <collision>
